Commit message: added lots of comments to read/write and updates ur5 urdf

File: ur10-replay/urdf/ur5e/ur5e_fixed.urdf (robot description, URDF)
Before this commit: robot ur5e, 9 links, 8 joints
Links:
- link base: geometry collision mesh filename=meshes/ur5e/collision/base.stl; visual mesh filename=meshes/ur5e/visual/base.dae
- link forearm_link: geometry collision mesh filename=meshes/ur5e/collision/forearm.stl; visual mesh filename=meshes/ur5e/visual/forearm.dae
- link shoulder_link: geometry collision mesh filename=meshes/ur5e/collision/shoulder.stl; visual mesh filename=meshes/ur5e/visual/shoulder.dae
- link upper_arm_link: geometry collision mesh filename=meshes/ur5e/collision/upperarm.stl; visual mesh filename=meshes/ur5e/visual/upperarm.dae
- link wrist_1_link: geometry collision mesh filename=meshes/ur5e/collision/wrist1.stl; visual mesh filename=meshes/ur5e/visual/wrist1.dae
- link wrist_2_link: geometry collision mesh filename=meshes/ur5e/collision/wrist2.stl; visual mesh filename=meshes/ur5e/visual/wrist2.dae
- link wrist_3_link: geometry collision mesh filename=meshes/ur5e/collision/wrist3.stl; visual mesh filename=meshes/ur5e/visual/wrist3.dae
Joints:
- joint elbow_joint: limit lower=-3.14159265359 upper=3.14159265359 effort=150.0 velocity=3.14 -> lower=-3.14159265359 upper=3.14159265359 effort=150.0 velocity=3.15; origin xyz=0 -0.1197 0.425 rpy=0 0 0 -> xyz=0 -0.131 0.425 rpy=0 0 0
- joint shoulder_lift_joint: limit lower=-6.2832 upper=6.2832 effort=150.0 velocity=3.14 -> lower=-6.28318530718 upper=6.28318530718 effort=150.0 velocity=3.15; origin xyz=0 0.13850 0 rpy=0 1.57079632679 0 -> xyz=0 0.138 0 rpy=0 1.57079632679 0
- joint shoulder_pan_joint: limit lower=-6.2832 upper=6.2832 effort=150.0 velocity=3.14 -> lower=-6.28318530718 upper=6.28318530718 effort=150.0 velocity=3.15; origin xyz=0 0 0.1625 rpy=0 0 0 -> xyz=0 0 0.163 rpy=0 0 0
- joint wrist_1_joint: axis 0 0 1 -> 0 1 0; limit lower=-6.2832 upper=6.2832 effort=28.0 velocity=6.28 -> lower=-6.28318530718 upper=6.28318530718 effort=28.0 velocity=3.2; origin xyz=0 0 0.3923 rpy=0 1.57079632679 0 -> xyz=0 0 0.392 rpy=0 1.57079632679 0
- joint wrist_2_joint: limit lower=-6.2832 upper=6.2832 effort=28.0 velocity=6.28 -> lower=-6.28318530718 upper=6.28318530718 effort=28.0 velocity=3.2; origin xyz=0 0.09465 0 rpy=0 0 0 -> xyz=0 0.127 0 rpy=0 0 0
- joint wrist_3_joint: axis 0 0 1 -> 0 1 0; limit lower=-6.2832 upper=6.2832 effort=28.0 velocity=6.28 -> lower=-6.28318530718 upper=6.28318530718 effort=28.0 velocity=3.2; origin xyz=0 0 0.09465 rpy=0 0 0 -> xyz=0 0 0.100 rpy=0 0 0
